File: KiCad/untitled.kicad_sch (KiCad schematic)
At the start: 20 parts, among them J2 Conn_01x03, J3 Conn_01x05, J5 DE9_Pins, SW1 SW_DPST_x2, Y1 8MHz, Y2 8MHz

Commit message: Part Micro quasi completat, falta afegir etiquetes de potencia
Parts:
- added J6: Conn_01x04, symbol Connector_Generic:Conn_01x04
- added R2, R3, R4, R5: 22k, symbol Device:R
- added SW1, SW2, SW3, SW4: SW_Push, symbol Switch:SW_Push
- C1: renamed from C7; value 100n -> 10u
- SWR: renamed from SW1; value SW_DPST_x2 -> SW_RESET
Connections:
- net GND: now also PIC32MX250F128B-50I/SO.27 (AVSS), SW1.1, SW2.1, SW3.1, SW4.1
- net RXD: no longer PIC32MX250F128B-50I/SO.7 (RB3)
- net SCLK: now also PIC32MX250F128B-50I/SO.4 (RB0); no longer PIC32MX250F128B-50I/SO.25 (RB14)
- net SDATA: now also PIC32MX250F128B-50I/SO.5 (RB1)
- net TXD: no longer PIC32MX250F128B-50I/SO.6 (RB2)
- net Vcc: now also R2.2, R3.2, R4.2, R5.2, SW1.2, SW2.2, SW3.2, SW4.2
- net CS_M1: now reaches PIC32MX250F128B-50I/SO.11 (RB4)
- net CS_M2: now reaches PIC32MX250F128B-50I/SO.12 (RA4)
- net CS_Hall: now reaches PIC32MX250F128B-50I/SO.14 (RB5)
- net CS_C1: now reaches PIC32MX250F128B-50I/SO.16 (RB7)
- net Boto 1: now reaches PIC32MX250F128B-50I/SO.2 (RA0)
- net Boto 4: now reaches PIC32MX250F128B-50I/SO.24 (RB13)
- net Boto 3: now reaches PIC32MX250F128B-50I/SO.26 (RB15)
- net Boto 2: now reaches PIC32MX250F128B-50I/SO.3 (RA1)
- new net: J6.1 (Pin_1), R5.1
- new net: J6.2 (Pin_2), R4.1
- new net: J6.3 (Pin_3), R3.1
- new net: J6.4 (Pin_4), R2.1
- new net SCLK1: PIC32MX250F128B-50I/SO.25 (RB14)
- no-connect marks 19 -> 8
Other:
- moved on the sheet: C12, C5, C6, C8, C9, FB5, J2, J3, R1, SWRA, Y1
