File: KiCad/Potencia.kicad_sch (KiCad schematic)
At the start: 2 parts, among them J4 Conn_01x08, U2 DRV8906QPWPRQ1

Commit message: Part Micro quasi completat, falta afegir etiquetes de potencia
Parts:
- added U1: BTS7004-1EPP, Package_SO:Infineon_PG-TSDSO-14-22, symbol Power_Management:BTS7004-1EPP
Connections:
- new net: U1.10 (OUT), U1.12 (OUT), U1.13 (OUT), U1.14 (OUT), U1.8 (OUT), U1.9 (OUT)
Changed lines of the file:
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@@
 	(wire
 		(pts
-			(xy 34.29 39.37) (xy 34.29 31.75)
+			(xy 34.29 39.37) (xy 34.29 26.67)
 		)
 		(stroke
@@
 	(wire
 		(pts
-			(xy 34.29 31.75) (xy 95.25 31.75)
+			(xy 34.29 26.67) (xy 95.25 26.67)
 		)
 		(stroke
@@
 	(wire
 		(pts
-			(xy 95.25 31.75) (xy 95.25 39.37)
+			(xy 95.25 26.67) (xy 95.25 39.37)
 		)
 		(stroke
@@
 					(unit 1)
 				)
+			)
+		)
+	)
+	(symbol
+		(lib_id "Power_Management:BTS7004-1EPP")
+		(at 142.24 68.58 0)
+		(unit 1)
+		(exclude_from_sim no)
+		(in_bom yes)
+		(on_board yes)
+		(dnp no)
+		(fields_autoplaced yes)
+		(property "Reference" "U1"
+			(at 156.21 62.1598 0)
+			(effects
+				(font
+					(size 1.27 1.27)
+				)
+			)
+		)
+		(property "Value" "BTS7004-1EPP"
+			(at 156.21 64.6998 0)
+			(effects
+				(font
+					(size 1.27 1.27)
+				)
+			)
+		)
+		(property "Footprint" "Package_SO:Infineon_PG-TSDSO-14-22"
+			(at 119.38 74.93 0)
+			(effects
+				(font
+					(size 1.27 1.27)
+				)
+				(hide yes)
+			)
+		)
+		(property "Datasheet" "https://www.infineon.com/dgdl/Infineon-BTS7004-1EPP-DS-v01_00-EN.pdf?fileId=5546d4626102d35a016147550a725555"
+			(at 142.24 81.28 0)
+			(effects
+				(font
+					(size 1.27 1.27)
+				)
+				(hide yes)
+			)
+		)
+		(property "Description" "Smart High-Side Power Switch, PROFET, One Channel, 12V, 15A, Rds(on) 4.4mΩ, PG-TSDSO-14-22"
+			(at 142.24 68.58 0)
+			(effects
+				(font
+					(size 1.27 1.27)
+				)
+				(hide yes)
+			)
+		)
+		(pin "4"
+		)
+		(pin "1"
+		)
+		(pin "6"
+		)
+		(pin "2"
+		)
+		(pin "3"
+		)
+		(pin "15"
+		)
+		(pin "5"
+		)
+		(pin "7"
+		)
+		(pin "11"
+		)
+		(pin "10"
+		)
+		(pin "12"
+		)
+		(pin "14"
+		)
+		(pin "8"
+		)
+		(pin "9"
+		)
+		(pin "13"
+		)
+		(instances
+			(project "Retrovisors_Carlos_Soler_Ingrid_Lopez"
+				(path "/a9cf8edd-cd44-4958-b775-951afc8c27af/9be4c8d4-69f1-4b7b-adb7-2777fc124923"
+					(reference "U1")
+					(unit 1)
+				)

Commit message: Microprocessador finalissim + placement de alimentacion y micro
Parts:
- J4: footprint (none) -> Connector_PinHeader_2.54mm:PinHeader_1x08_P2.54mm_Vertical
- U2: footprint HTSSOP24_PWP_TEX -> Driver_m:HTSSOP24_PWP_TEX
Changed lines of the file:
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@@
 			)
 		)
-		(property "Footprint" "HTSSOP24_PWP_TEX"
+		(property "Footprint" "Driver_m:HTSSOP24_PWP_TEX"
 			(at 34.29 39.37 0)
 			(effects
@@
 			)
 		)
-		(property "Footprint" ""
+		(property "Footprint" "Connector_PinHeader_2.54mm:PinHeader_1x08_P2.54mm_Vertical"
 			(at 127 35.56 0)
 			(effects
