File: KiCad/Digital.kicad_sch (KiCad schematic)
At the start: 39 parts, among them IC1 PIC24H, J2 DE9_Plug_MountingHoles, J3 DE9_Plug_MountingHoles, J4 Conn_01x03, J7 Conn_01x05, SW1 SW_DP3T, SW2 SW_DP3T, SW3 SW_DP3T, SW4 OP/CL, SW7 OP/CL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

Commit message: pcb definitiva
Connections:
- net DLX_D: now also U3.9 (P4); no longer U3.12 (P7)
- net DRX_U: now also U3.12 (P7); no longer U3.9 (P4)
- net ConMu: now reaches J4.1 (Pin_1), J7.3 (Pin_3)
- net RM_BO: now reaches R5.1, R6.2, SW1.1
- net SP: now reaches IC1.11 (RC0/T1OSO/T13CKI), R35.1, SW7.2
- net SCL: now reaches IC1.14 (RC3/SCK/SCL), R43.1, TP2.1, U3.14 (SCL)
- net SDA: now reaches IC1.15 (RC4/SDI/SDA), R44.1, TP1.1, U3.15 (SDA)
- net AL1: now reaches IC1.2 (RA0/AN0), R31.2, R32.1
- net AL2: now reaches IC1.3 (RA1/AN1), R33.2, R34.1
- net RS: now reaches R29.1, U2.8 (Rs)
- net SE_BO: now reaches R8.1, R9.2, SW3.1
- net LM_BO: now reaches R2.1, R3.2, SW2.1
- net osc1 renamed OSC1
- net osc2 renamed OSC2
Other:
- note added: "25/05/2026"
- note added: "Aqui podem veure el microcontrolador y les seves conexions, tambe esta la botonera per tal de poder moure els retrovisors."
- note added: "Etapa Digital"
- moved on the sheet: SW7
