File: KiCad/Digital.kicad_sch (KiCad schematic)
At the start: 39 parts, among them IC1 PIC24H, J2 DE9_Plug_MountingHoles, J3 DE9_Plug_MountingHoles, J4 Conn_01x03, J7 Conn_01x05, SW1 SW_DP3T, SW2 SW_DP3T, SW3 SW_DP3T, SW4 OP/CL, SW7 OP/CL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

Commit message: afegit tot final
Other:
- note added: "S'observa el microcontrolador i les seves conexions, amb la corresponent botonera per tal de poder moure els retrovisors."
- note removed: "Aqui podem veure el microcontrolador y les seves conexions, tambe esta la botonera per tal de poder moure els retrovisors."
- moved on the sheet: C3, C4, C5, IC1, J3, J4, J7, R1, R10, R2, R3, R31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
