File: KiCad/Retrovisors_Carlos_Soler_Ingrid_Lopez.kicad_sch (KiCad schematic)
At the start: 0 parts

Commit message: Creacio de branca nova i update
Parts:
- added C1: 100n, Capacitor_SMD:C_0603_1608Metric_Pad1.08x0.95mm_HandSolder, symbol Device:C
- added C2: 100n, Capacitor_SMD:C_0805_2012Metric, symbol Device:C
- added C3, C4: 22p, Capacitor_SMD:C_0805_2012Metric_Pad1.18x1.45mm_HandSolder, symbol Device:C
- added C5: 10n, Capacitor_SMD:C_0805_2012Metric_Pad1.18x1.45mm_HandSolder, symbol Device:C
- added C6: 100n, Capacitor_SMD:C_0805_2012Metric_Pad1.18x1.45mm_HandSolder, symbol Device:C
- added C_Polarized_1: 220uF, Capacitor_THT:C_Radial_D4.0mm_H5.0mm_P1.50mm, symbol Device:C_Polarized_Small_US
- added C_Polarized_2: 10uF, Capacitor_THT:C_Radial_D4.0mm_H5.0mm_P1.50mm, symbol Device:C_Polarized_Small_US
- added D1: SM6T36A, Diode_SMD:D_SMB, symbol Diode:SM6T36A
- added D10, D11, D12, D13, D3, D4, D5, D6, D8, D9: 1N4002, Diode_THT:D_DO-41_SOD81_P10.16mm_Horizontal, symbol Device:D
- added D14: LED, symbol Device:LED
- added D2: LED, LED_SMD:LED_0805_2012Metric, symbol Device:LED
- added D7: FS1G-LTP, FS1G:DIOM5226X244N, symbol FS1G-LTP:FS1G-LTP
- added FB1: FerriteBead_Small, BLM15BB050SZ1D:BEADC1005X55N, symbol Device:FerriteBead_Small
- added IC1: PIC24H, PIC18F258-I_SO:SOIC127P1030X265-28N, symbol PIC18F2580-I_SO:PIC18F2580-I_SO
- added J1: Conn_01x02_Pin, Connector_PinHeader_2.54mm:PinHeader_1x02_P2.54mm_Vertical, symbol Connector:Conn_01x02_Pin
- added J10, J5, J6, J8, J9: Conn_01x02, Connector_PinHeader_2.54mm:PinHeader_1x02_P2.54mm_Vertical, symbol Connector_Generic:Conn_01x02
- added J11, J12: Conn_01x02, symbol Connector_Generic:Conn_01x02
- added J2, J3: DE9_Plug_MountingHoles, Connector_Dsub:DSUB-9_Female_Vertical_P2.77x2.84mm_MountingHoles, symbol Connector:DE9_Plug_MountingHoles
- added J4: Conn_01x03, Connector_PinHeader_2.54mm:PinHeader_1x03_P2.54mm_Vertical, symbol Connector_Generic:Conn_01x03
- added J7: Conn_01x05, Connector_PinHeader_2.54mm:PinHeader_1x05_P2.54mm_Vertical, symbol Connector_Generic:Conn_01x05
- added K1, K10, K2, K3, K4, K5, K6, K7, K8, K9: G6E, Relay_THT:Relay_SPDT_Omron_G6E, symbol Relay:G6E
- added Q1, Q10, Q2, Q3, Q4, Q5, Q6, Q7, Q8, Q9: NMOS, CSD19505KCS:TO254P470X1016X1965-3P, symbol Simulation_SPICE:NMOS
- added Q11, Q12: IRLZ44N, Package_TO_SOT_THT:TO-220-3_Vertical, symbol Transistor_FET:IRLZ44N
- added R1: 1k, Resistor_SMD:R_1206_3216Metric_Pad1.30x1.75mm_HandSolder, symbol Device:R
- added R10, R11, R12, R13, R14, R15, R16, R17, R18, R19, R2, R20, R4, R7, R8, R9: 10k, Resistor_SMD:R_1206_3216Metric_Pad1.30x1.75mm_HandSolder, symbol Device:R
- added R21, R22, R27, R28: 10k, symbol Device:R
- added R23: 330, symbol Device:R
- added R26: R, symbol Device:R
- added R3: 60, Resistor_SMD:R_1206_3216Metric_Pad1.30x1.75mm_HandSolder, symbol Device:R
- added R5, R6: 4.7k, Resistor_SMD:R_1206_3216Metric_Pad1.30x1.75mm_HandSolder, symbol Device:R
- added S1, S2: 2-1437565-7, 2-1437565-7:SW_2-1437565-7, symbol 2-1437565-7:2-1437565-7
- added SW1, SW2, SW3: SW_DP3T, Button_Switch_THT:SW_DIP_SPSTx02_Piano_10.8x6.64mm_W7.62mm_P2.54mm, symbol Switch:SW_DP3T
- added U2: MCP2551-I-SN, Package_SO:SOIC-8_3.9x4.9mm_P1.27mm, symbol Interface_CAN_LIN:MCP2551-I-SN
- added U3: L78S05CV, Package_TO_SOT_THT:TO-220-3_Horizontal_TabDown, symbol Regulator_Linear:LT1117-5.0
- added Y1: Crystal, Crystal:Crystal_SMD_Abracon_ABM3-2Pin_5.0x3.2mm_HandSoldering, symbol Device:Crystal
Connections:
- new net: J4.1 (Pin_1), J7.3 (Pin_3)
- new net: D11.1 (K), K8.1
- new net: R11.2, R9.1, SW1.1
- new net: Q12.1 (G), R27.2, R28.1
- new net: Q11.1 (G), R21.2, R22.1
- new net: J11.2 (Pin_2), Q11.2 (D)
- new net: C4.1, IC1.10 (OSC2/CLKO/RA6), Y1.2
- new net: IC1.15 (RC4/SDI/SDA), R23.1
- new net: IC1.4 (RA2/AN2/VREF-), S2.1, S2.2
- new net: C3.1, IC1.9 (OSC1/CLKI/RA7), Y1.1
- new net: R6.1, U2.8 (Rs)
- new net: J4.3 (Pin_3), R5.2, S1.1, S1.2
- new net: R19.1, R20.2, SW3.1
- new net: R17.1, R18.2, SW2.1
- new net: J12.2 (Pin_2), Q12.2 (D)
- new net: D9.1 (K), K4.1
- new net: D2.2 (A), R1.2
- new net: D14.2 (A), R23.2
- new net +12V: D7.2 (A), J1.1 (Pin_1)
- new net CAL_L: IC1.26 (RB5/KBI1/PGM), R21.1
- new net CAL_R: IC1.16 (RC5/SDO), R27.1
- new net CAN+: J2.7, R3.1, U2.7 (CANH)
- new net CAN-: J2.2, R3.2, U2.6 (CANL)
- new net CANRX: IC1.24 (RB3/CANRX), U2.4 (RXD)
- new net CANTX: IC1.23 (RB2/INT2/CANTX), U2.1 (TXD)
- new net DLX_D: IC1.6 (RA4/T0CKI), Q2.2 (G), R12.1
- new net DLX_U: IC1.5 (RA3/AN3/VREF+), Q1.2 (G), R10.1
- new net DLY_D: IC1.3 (RA1/AN1), Q6.2 (G), R16.1
- new net DLY_U: IC1.2 (RA0/AN0), Q5.2 (G), R14.2
- new net DM_C: IC1.12 (RC1/T1OSI), Q10.2 (G), R15.1
- new net DM_O: IC1.11 (RC0/T1OSO/T13CKI), Q9.2 (G), R13.1
- new net DRX_D: Q7.2 (G), R7.1
- new net DRX_U: Q3.2 (G), R2.1
- new net DRY_D: Q8.2 (G), R8.1
- new net DRY_U: Q4.2 (G), R4.2
- new net GND: C2.2, C3.2, C4.2, C5.2, C6.1, C_Polarized_2.2, D14.1 (K), D2.1 (K), FB1.2, IC1.19 (VSS_2), IC1.8 (VSS_1), J2.6, J3.5, J7.1 (Pin_1), Q11.3 (S), Q12.3 (S), R10.2, R11.1, R12.2, R13.2, R14.1, R15.2, R16.2, R18.1, R2.2, R20.1, R22.2, R26.2, R28.2, R4.1, R6.2, R7.2, R8.2, S1.3, S1.4, S2.3, S2.4, SW1.2, SW2.2, SW3.2, U2.2 (VSS)
- new net GNDPWR: C1.2, C_Polarized_1.2, D1.2 (A2), FB1.1, J1.2 (Pin_2), K1.10, K10.10, K2.10, K3.10, K4.10, K5.10, K6.10, K7.10, K8.10, K9.10, Q1.3 (S), Q10.3 (S), Q2.3 (S), Q3.3 (S), Q4.3 (S), Q5.3 (S), Q6.3 (S), Q7.3 (S), Q8.3 (S), Q9.3 (S), U3.1 (GND), U3.4 (GND)
- new net LM_button: IC1.25 (RB4/KBI0/AN9), SW2.3
- new net MCLR: IC1.1 (~{MCLR}/VPP/RE3), J4.2 (Pin_2)
- new net MLX_D: J5.2 (Pin_2), K2.7
- new net MLX_U: J5.1 (Pin_1), K1.7
- new net MLY_D: J6.2 (Pin_2), K6.7
- new net MLY_U: J6.1 (Pin_1), K5.7
- new net MM_C: J10.2 (Pin_2), K10.7
- new net MM_O: J10.1 (Pin_1), K9.7
- new net MRX_D: J9.2 (Pin_2), K7.7
- new net MRX_U: J9.1 (Pin_1), K3.7
- new net MRY_D: J8.2 (Pin_2), K8.7
- new net MRY_U: J8.1 (Pin_1), K4.7
- new net RM_button: IC1.21 (RB0/INT0/AN10), R26.1, SW1.3
- new net RX: IC1.18 (RC7/RX/DT), J3.2
- new net SCLK: IC1.27 (RB6/KBI2/PGC), J7.4 (Pin_4)
- new net SDATA: IC1.28 (RB7/KBI3/PGD), J7.5 (Pin_5)
- new net TX: IC1.17 (RC6/TX/CK), J3.3
- new net VBAT_PROT: C1.1, C_Polarized_1.1, D1.1 (A1), D10.1 (K), D12.1 (K), D13.1 (K), D3.1 (K), D4.1 (K), D5.1 (K), D6.1 (K), D7.1 (K), D8.1 (K), J11.1 (Pin_1), J12.1 (Pin_1), K1.1, K1.12, K10.1, K10.12, K2.1, K2.12, K3.1, K3.12, K4.12, K5.1, K5.12, K6.1, K6.12, K7.1, K7.12, K8.12, K9.1, K9.12, U3.3 (VI)
- new net VCC: C2.1, C5.1, C6.2, C_Polarized_2.1, IC1.20 (VDD), J7.2 (Pin_2), R1.1, R17.2, R19.2, R5.1, R9.2, SW1.4, SW2.4, SW3.4, U2.3 (VDD), U3.2 (VO)
- new net Vdrain1: D12.2 (A), D5.2 (A), D8.2 (A), K1.6, K3.6, K9.6, Q1.1 (D), Q3.1 (D), Q9.1 (D)
- new net Vdrain2: D10.2 (A), D13.2 (A), D6.2 (A), K10.6, K2.6, K7.6, Q10.1 (D), Q2.1 (D), Q7.1 (D)
- new net Vdrain3: D11.2 (A), D4.2 (A), K6.6, K8.6, Q6.1 (D), Q8.1 (D)
- new net Vdrain4: D3.2 (A), D9.2 (A), K4.6, K5.6, Q4.1 (D), Q5.1 (D)
- new net select_button: IC1.22 (RB1/INT1/AN8), SW3.3
- no-connect marks 0 -> 16
Other:
- removed sheet Alimentació
- removed sheet Digital
- removed sheet Potencia
- note added: "25/05/2026"
- note added: "BOTONERA"
- note added: "BUS CAN"
- note added: "CALEFACTOR"
- note added: "CRISTALL"
- note added: "DRIVER DEL MOTOR DE L'EIX X"
- note added: "DRIVER DEL MOTOR DE L'EIX Y"
- note added: "DRIVER DEL MOTOR DE OBRIR I TENCAR"
- note added: "ESQUEMÀTIC RETROVISORS D'UN COTXE"
- note added: "INPUTS"
- note added: "Ingrid Lopez Carlos Soler"
- note added: "MICROCONTROLADOR"
- note added: "REGULADOR DE TENSIÓ"
- note added: "USART"

Commit message: actualització (NO VERSIÓ FINAL)
Parts:
- added C7: 100n, Capacitor_SMD:C_0805_2012Metric_Pad1.18x1.45mm_HandSolder, symbol Device:C
- added R24, R25, R29, R30: 10k, Resistor_SMD:R_1206_3216Metric_Pad1.30x1.75mm_HandSolder, symbol Device:R
- added R31: 1k, Resistor_SMD:R_1206_3216Metric_Pad1.30x1.75mm_HandSolder, symbol Device:R
- added R32: 2,5k, Resistor_SMD:R_1206_3216Metric_Pad1.30x1.75mm_HandSolder, symbol Device:R
- added R33: 5k, Resistor_SMD:R_1206_3216Metric_Pad1.30x1.75mm_HandSolder, symbol Device:R
- added R_Shunt1: 5, Resistor_SMD:R_Shunt_Ohmite_LVK12, symbol Device:R_Shunt
- added U4, U5: ${SIM.PARAMS}, SOT95P280X145-5N:SOT95P280X145-5N, symbol Simulation_SPICE:OPAMP
Connections:
- net GND: now also C7.2, R29.1, R_Shunt1.4, U4.5 (V-)
- net GNDPWR: no longer K10.10, K9.10
- net VCC: now also C7.1, R32.2, U4.4 (V+), U5.4 (V+)
- net SC_IN: now reaches IC1.14 (RC3/SCK/SCL)
- net SC_IN: now also U5.3
- new net: R24.1, R_Shunt1.2
- new net: R25.1, R_Shunt1.3
- new net: R32.1, R33.2, U5.2 (-)
- new net: R30.2, R31.1, U4.3, U5.1 (+)
- new net: R31.2, R33.1, U5.5 (V-)
- new net: R24.2, R30.1, U4.1 (+)
- new net: R25.2, R29.2, U4.2 (-)
- new net FI_MOTOR: K10.10, K9.10, R_Shunt1.1
Other:
- note added: "LED uC"
- note added: "SENSOR DE CORRENT DE FINAL DE CARRERA"
- moved on the sheet: K10

Commit message: esquematic + placement (FALTA ROUTING DELS DRIVERS!!)
Parts:
- removed C1: 100n, Capacitor_SMD:C_0603_1608Metric_Pad1.08x0.95mm_HandSolder, symbol Device:C
- removed C_Polarized_1: 220uF, Capacitor_THT:C_Radial_D4.0mm_H5.0mm_P1.50mm, symbol Device:C_Polarized_Small_US
- removed C_Polarized_2: 10uF, Capacitor_THT:C_Radial_D4.0mm_H5.0mm_P1.50mm, symbol Device:C_Polarized_Small_US
- removed D1: SM6T36A, Diode_SMD:D_SMB, symbol Diode:SM6T36A
- removed D14: LED, symbol Device:LED
- removed D7: FS1G-LTP, FS1G:DIOM5226X244N, symbol FS1G-LTP:FS1G-LTP
- removed FB1: FerriteBead_Small, BLM15BB050SZ1D:BEADC1005X55N, symbol Device:FerriteBead_Small
- removed J1: Conn_01x02_Pin, Connector_PinHeader_2.54mm:PinHeader_1x02_P2.54mm_Vertical, symbol Connector:Conn_01x02_Pin
- removed R1: 1k, Resistor_SMD:R_1206_3216Metric_Pad1.30x1.75mm_HandSolder, symbol Device:R
- removed R23: 330, symbol Device:R
- removed S1, S2: 2-1437565-7, 2-1437565-7:SW_2-1437565-7, symbol 2-1437565-7:2-1437565-7
- removed U3: L78S05CV, Package_TO_SOT_THT:TO-220-3_Horizontal_TabDown, symbol Regulator_Linear:LT1117-5.0
- added C1, C10, C13, C9: 1u, Capacitor_SMD:CP_Elec_4x5.7, symbol Device:C_Polarized
- added C11, C12, C8: 100n, Capacitor_SMD:C_0805_2012Metric_Pad1.18x1.45mm_HandSolder, symbol Device:C
- added D1, D7: G_LED, LED_SMD:LED_0805_2012Metric_Pad1.15x1.40mm_HandSolder, symbol Device:LED
- added D15: FS1G-LTP, AA_footprints:DIOM5225X244N, symbol FS1G-LTP:FS1G-LTP
- added D16: D_transil, Diode_THT:D_DO-35_SOD27_P2.54mm_Vertical_AnodeUp, symbol Device:D_Zener
- added J14: Conn_01x02_Pin, Connector_PinHeader_2.54mm:PinHeader_1x02_P2.54mm_Vertical, symbol Connector:Conn_01x02_Pin
- added R10, R28, R4: 220, Resistor_SMD:R_1206_3216Metric_Pad1.30x1.75mm_HandSolder, symbol Device:R
- added R25: 150, Resistor_SMD:R_0805_2012Metric_Pad1.20x1.40mm_HandSolder, symbol Device:R
- added R26, R27: 1k, Resistor_SMD:R_1206_3216Metric_Pad1.30x1.75mm_HandSolder, symbol Device:R
- added R31, R33: LDR07, OptoDevice:R_LDR_5.1x4.3mm_P3.4mm_Vertical, symbol Sensor_Optical:LDR07
- added R32, R34, R35: 10k, Resistor_SMD:R_1206_3216Metric_Pad1.30x1.75mm_HandSolder, symbol Device:R
- added SW4, SW7: OP/CL, Button_Switch_SMD:SW_SPST_PTS647_Sx38, symbol Switch:SW_Push
- added U1: TSR0.5-2450, Converter_DCDC:Converter_DCDC_TRACO_TSR0.5-24xx_TSR0.5-24xxx_THT, symbol Converter_DCDC:TSR0.5-2450
- added U6: LM1117DT-3.3, Package_TO_SOT_SMD:TO-252-3_TabPin2, symbol Regulator_Linear:LM1117DT-3.3
- C2: footprint Capacitor_SMD:C_0805_2012Metric -> Capacitor_SMD:C_0805_2012Metric_Pad1.18x1.45mm_HandSolder
- D2: value LED -> G_LED; footprint LED_SMD:LED_0805_2012Metric -> LED_SMD:LED_0805_2012Metric_Pad1.15x1.40mm_HandSolder; LSCS (none) -> C125090
- IC1: footprint PIC18F258-I_SO:SOIC127P1030X265-28N -> AA_footprints:SOIC127P1030X265-28N
- J11, J12: footprint (none) -> Connector_PinHeader_2.54mm:PinHeader_1x02_P2.54mm_Vertical
- J2, J3: footprint Connector_Dsub:DSUB-9_Female_Vertical_P2.77x2.84mm_MountingHoles -> AA_footprints:DSUB-9_Female_Vertical_Pitch2.77x2.84mm_MountingHoles
- Q1, Q10, Q2, Q8, Q9: footprint CSD19505KCS:TO254P470X1016X1965-3P -> AA_footprints:TO254P470X1016X1965-3P
- Q3: renamed from Q5; footprint CSD19505KCS:TO254P470X1016X1965-3P -> AA_footprints:TO254P470X1016X1965-3P
- Q4: renamed from Q6; footprint CSD19505KCS:TO254P470X1016X1965-3P -> AA_footprints:TO254P470X1016X1965-3P
- Q5: renamed from Q3; footprint CSD19505KCS:TO254P470X1016X1965-3P -> AA_footprints:TO254P470X1016X1965-3P
- Q6: renamed from Q7; footprint CSD19505KCS:TO254P470X1016X1965-3P -> AA_footprints:TO254P470X1016X1965-3P
- Q7: renamed from Q4; footprint CSD19505KCS:TO254P470X1016X1965-3P -> AA_footprints:TO254P470X1016X1965-3P
- R21, R22: footprint (none) -> Resistor_SMD:R_1206_3216Metric_Pad1.30x1.75mm_HandSolder
- R23: renamed from R27; footprint (none) -> Resistor_SMD:R_1206_3216Metric_Pad1.30x1.75mm_HandSolder
- R24: renamed from R28; footprint (none) -> Resistor_SMD:R_1206_3216Metric_Pad1.30x1.75mm_HandSolder
- R7: renamed from R26; value R -> 220; footprint (none) -> Resistor_SMD:R_1206_3216Metric_Pad1.30x1.75mm_HandSolder
- U4, U5: footprint SOT95P280X145-5N:SOT95P280X145-5N -> AA_footprints:SOT95P280X145-5N
- renumbered J5 to J1, J6 to J3-4, J9 to J5, J8 to J7-8, J10 to J9, K5 to K3, K6 to K4, K3 to K5, K7 to K6, K4 to K7, R5 to R1, R14 to R11, R16 to R12, R10 to R13, R12 to R14, R4 to R15, R8 to R16, R2 to R17, R7 to R18, R13 to R19, R17 to R2, R15 to R20, R6 to R29, R18 to R3, R3 to R30, R24 to R36, R25 to R37, R30 to R38, R29 to R39, R31 to R40, R32 to R41, R33 to R42, R9 to R5, R11 to R6, R19 to R8, R20 to R9
Connections:
- net +12V: now also D15.2 (A), J14.1 (Pin_1)
- net DLX_D: now also IC1.7 (RA5/AN4/~{SS}/HLVDIN); no longer IC1.6 (RA4/T0CKI)
- net DLX_U: now also IC1.6 (RA4/T0CKI); no longer IC1.5 (RA3/AN3/VREF+)
- net GND: now also C1.2, C10.2, C11.2, C12.2, C13.2, D1.1 (K), R10.2, R27.2, R32.2, R34.2, R35.2, R4.2, SW4.2, U6.1 (GND); no longer D2.1 (K)
- net GNDPWR: now also C8.2, C9.2, D16.2 (A), J14.2 (Pin_2), U1.2 (GND)
- net LM_button: now also R4.1
- net SC_IN: now also IC1.15 (RC4/SDI/SDA); no longer IC1.14 (RC3/SCK/SCL)
- net VBAT_PROT: now also D11.1 (K), D9.1 (K), K7.1, K8.1, C8.1, C9.1, D15.1 (K), D16.1 (K), U1.1 (Vin)
- net VCC: now also C1.1, R25.1, R26.1, R31.1, R33.1, SW7.1, U6.2 (VO)
- net reset: now also J4.3 (Pin_3), R1.2, SW4.1
- net select_button: now also R10.1
- net angle_m: now reaches IC1.13 (RC2/CCP1)
- net angle_m: now also R28.2
- net at IC1.4 (RA2/AN2/VREF-): now also R31.2, R32.1
- net at D2.2 (A): now also D7.1 (K), R26.2, R27.1
- new net: D2.1 (K), D7.2 (A), R28.1
- new net: IC1.14 (RC3/SCK/SCL), R35.1, SW7.2
- new net: IC1.5 (RA3/AN3/VREF+), R33.2, R34.1
- new net: C10.1, C11.1, C12.1, C13.1, U1.3 (Vout), U6.3 (VI)
- new net: D1.2 (A), R25.2
- no-connect marks 16 -> 15
Other:
- note added: "CALEFACTORS"
- note added: "LDR'S ANTI-ENLLUERNAMENT"
- note added: "LEDS SENSOR ANGLE MORT"
- note added: "Led per a verificar que hi ha corrent."
- note added: "SW OPEN/CLOSE"
- note removed: "CALEFACTOR"
- note removed: "LED uC"
- moved on the sheet: C3, C4, C5, C6, C7, D10, D11, D12, D13, D5, D6, D8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

Commit message: Modificació placement
Connections:
- net CAL_L: now also J11.2 (Pin_2), Q11.2 (D)
- net CAL_R: now also J12.2 (Pin_2), Q12.2 (D)
- net CANRX: now also IC1.23 (RB3/CANRX); no longer IC1.24 (RB3/CANRX)
- net CANTX: now also IC1.24 (RB2/INT2/CANTX); no longer IC1.23 (RB2/INT2/CANTX)
Changed lines of the file:
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@@
 	(wire
 		(pts
+			(xy 306.07 223.52) (xy 311.15 223.52)
+		)
+		(stroke
+			(width 0)
+			(type default)
+		)
+	)
+	(wire
+		(pts
 			(xy 320.548 145.542) (xy 318.516 145.542)
 		)
@@
 	(wire
 		(pts
-			(xy 134.112 157.48) (xy 132.08 157.48)
+			(xy 134.62 157.48) (xy 132.08 157.48)
 		)
 		(stroke
@@
 	(wire
 		(pts
-			(xy 302.387 231.14) (xy 302.387 237.998)
+			(xy 302.26 231.14) (xy 302.26 237.998)
 		)
 		(stroke
@@
 	(wire
 		(pts
-			(xy 302.387 217.678) (xy 302.387 220.98)
-		)
-		(stroke
-			(width 0)
-			(type default)
-		)
-	)
-	(wire
-		(pts
 			(xy 227.33 207.01) (xy 227.33 208.28)
 		)
@@
 	(wire
 		(pts
-			(xy 306.197 228.6) (xy 311.277 228.6)
+			(xy 306.07 228.6) (xy 311.15 228.6)
 		)
 		(stroke
@@
 	(wire
 		(pts
-			(xy 318.897 228.6) (xy 323.723 228.6)
+			(xy 318.77 228.6) (xy 323.723 228.6)
 		)
 		(stroke
@@
 	(wire
 		(pts
-			(xy 318.516 223.52) (xy 324.612 223.52)
+			(xy 318.77 223.52) (xy 324.612 223.52)
 		)
 		(stroke
@@
 	(wire
 		(pts
+			(xy 300.99 217.17) (xy 302.26 217.17)
+		)
+		(stroke
+			(width 0)
+			(type default)
+		)
+	)
+	(wire
+		(pts
 			(xy 199.136 104.902) (xy 199.136 102.108)
 		)
@@
 	(wire
 		(pts
-			(xy 310.134 237.998) (xy 302.387 237.998)
+			(xy 310.134 237.998) (xy 302.26 237.998)
 		)
 		(stroke
@@
 	(wire
 		(pts
-			(xy 306.197 223.52) (xy 310.896 223.52)
+			(xy 302.26 217.17) (xy 302.26 220.98)
 		)
 		(stroke
@@
 	(wire
 		(pts
-			(xy 301.117 217.678) (xy 302.387 217.678)
-		)
-		(stroke
-			(width 0)
-			(type default)
-		)
-	)
-	(wire
-		(pts
 			(xy 223.52 18.796) (xy 236.982 18.796)
 		)
@@
 		)
 	)
+	(label "CAL_L"
+		(at 234.95 157.48 90)
+		(effects
+			(font
+				(size 1.27 1.27)
+			)
+			(justify left bottom)
+		)
+	)
 	(label "CAN+"
 		(at 62.738 103.886 0)
@@
 		)
 	)
+	(label "CAL_R"
+		(at 236.22 191.77 90)
+		(effects
+			(font
+				(size 1.27 1.27)
+			)
+			(justify left bottom)
+		)
+	)
 	(label "Vdrain3"
 		(at 250.952 42.418 0)
@@
 	(global_label "CANTX"
 		(shape bidirectional)
-		(at 134.112 157.48 0)
+		(at 134.62 157.48 0)
 		(fields_autoplaced yes)
 		(effects
@@
 		)
 		(property "Intersheetrefs" "${INTERSHEET_REFS}"
-			(at 143.9953 157.48 0)
+			(at 144.5033 157.48 0)
 			(effects
 				(font
@@
 	(global_label "FI_MOTOR"
 		(shape input)
-		(at 301.117 217.678 180)
+		(at 300.99 217.17 180)
 		(fields_autoplaced yes)
 		(effects
@@
 		)
 		(property "Intersheetrefs" "${INTERSHEET_REFS}"
-			(at 289.1208 217.678 0)
+			(at 288.9938 217.17 0)
 			(effects
 				(font
@@
 	(symbol
 		(lib_id "Device:R_Shunt")
-		(at 302.387 226.06 0)
+		(at 302.26 226.06 0)
 		(unit 1)
 		(exclude_from_sim no)
@@
 		(on_board yes)
 		(dnp no)
-		(fields_autoplaced yes)
 		(property "Reference" "R_Shunt1"
-			(at 300.228 225.425 0)
+			(at 300.101 225.425 0)
 			(effects
 				(font
@@
 		)
 		(property "Value" "5"
-			(at 300.228 227.965 0)
+			(at 300.101 227.965 0)
 			(effects
 				(font
@@
 		)
 		(property "Footprint" "Resistor_SMD:R_Shunt_Ohmite_LVK12"
-			(at 300.609 226.06 90)
+			(at 300.482 226.06 90)
 			(effects
 				(font
@@
 		)
 		(property "Datasheet" "~"
-			(at 302.387 226.06 0)
+			(at 302.26 226.06 0)
 			(effects
 				(font
@@
 		)
 		(property "Description" ""
-			(at 302.387 226.06 0)
+			(at 302.26 226.06 0)
 			(effects
 				(font
@@
 	(symbol
 		(lib_id "Device:R")
-		(at 315.087 228.6 90)
+		(at 314.96 228.6 90)
 		(unit 1)
 		(exclude_from_sim no)
@@
 		(dnp no)
 		(property "Reference" "R37"
-			(at 312.801 230.886 90)
+			(at 312.674 230.886 90)
 			(effects
 				(font
@@
 		)
 		(property "Value" "10k"
-			(at 317.627 230.759 90)
+			(at 317.5 230.759 90)
 			(effects
 				(font
@@
 		)
 		(property "Footprint" "Resistor_SMD:R_1206_3216Metric_Pad1.30x1.75mm_HandSolder"
-			(at 315.087 230.378 90)
+			(at 314.96 230.378 90)
 			(effects
 				(font
@@
 		)
 		(property "Datasheet" "~"
-			(at 315.087 228.6 0)
+			(at 314.96 228.6 0)
 			(effects
 				(font
@@
 		)
 		(property "Description" ""
-			(at 315.087 228.6 0)
+			(at 314.96 228.6 0)
 			(effects
 				(font
@@
 	(symbol
 		(lib_id "Device:R")
-		(at 314.706 223.52 90)
+		(at 314.96 223.52 90)
 		(unit 1)
 		(exclude_from_sim no)
@@
 		(dnp no)
 		(property "Reference" "R36"
-			(at 312.42 221.615 90)
+			(at 312.674 221.615 90)
 			(effects
 				(font
@@
 		)
 		(property "Value" "10k"
-			(at 317.754 221.615 90)
+			(at 318.008 221.615 90)
 			(effects
 				(font
@@
 		)
 		(property "Footprint" "Resistor_SMD:R_1206_3216Metric_Pad1.30x1.75mm_HandSolder"
-			(at 314.706 225.298 90)
+			(at 314.96 225.298 90)
 			(effects
 				(font
@@
 		)
 		(property "Datasheet" "~"
-			(at 314.706 223.52 0)
+			(at 314.96 223.52 0)
 			(effects
 				(font
@@
 		)
 		(property "Description" ""
-			(at 314.706 223.52 0)
+			(at 314.96 223.52 0)
 			(effects
 				(font
