File: KiCad/Retrovisors_Carlos_Soler_Ingrid_Lopez.kicad_sch (KiCad schematic)
At the start: 117 parts, among them IC1 PIC24H, J1 Conn_01x02, J11 Conn_01x02, J12 Conn_01x02, J14 Conn_01x02_Pin, J2 DE9_Plug_MountingHoles, J3 DE9_Plug_MountingHoles, J3-4 Conn_01x02, J4 Conn_01x03, J5 Conn_01x02, J7 Conn_01x05, J7-8 Conn_01x02, J9 Conn_01x02, K1 G6E, K10 G6E, K2 G6E, K3 G6E, K4 G6E, K5 G6E, K6 G6E, K7 G6E, K8 G6E, K9 G6E, Q1 NMOS, Q10 NMOS, Q11 IRLZ44N, Q12 IRLZ44N, Q2 NMOS, Q3 NMOS, Q4 NMOS, Q5 NMOS, Q6 NMOS, Q7 NMOS, Q8 NMOS, Q9 NMOS, SW1 SW_DP3T, SW2 SW_DP3T, SW3 SW_DP3T, SW4 OP/CL, SW7 OP/CL, U1 TSR0.5-2450, U2 MCP2551-I-SN, U4 ${SIM.PARAMS}, U5 ${SIM.PARAMS}, U6 LM1117DT-3.3, Y1 Crystal

Commit message: modificando todos los GND eliminamos GND PWR
Parts:
- removed C1, C10, C13, C9: 1u, Capacitor_SMD:CP_Elec_4x5.7, symbol Device:C_Polarized
- removed C11, C12, C2, C6, C7, C8: 100n, Capacitor_SMD:C_0805_2012Metric_Pad1.18x1.45mm_HandSolder, symbol Device:C
- removed C3, C4: 22p, Capacitor_SMD:C_0805_2012Metric_Pad1.18x1.45mm_HandSolder, symbol Device:C
- removed C5: 10n, Capacitor_SMD:C_0805_2012Metric_Pad1.18x1.45mm_HandSolder, symbol Device:C
- removed D1, D2, D7: G_LED, LED_SMD:LED_0805_2012Metric_Pad1.15x1.40mm_HandSolder, symbol Device:LED
- removed D10, D11, D12, D13, D3, D4, D5, D6, D8, D9: 1N4002, Diode_THT:D_DO-41_SOD81_P10.16mm_Horizontal, symbol Device:D
- removed D15: FS1G-LTP, AA_footprints:DIOM5225X244N, symbol FS1G-LTP:FS1G-LTP
- removed D16: D_transil, Diode_THT:D_DO-35_SOD27_P2.54mm_Vertical_AnodeUp, symbol Device:D_Zener
- removed IC1: PIC24H, AA_footprints:SOIC127P1030X265-28N, symbol PIC18F2580-I_SO:PIC18F2580-I_SO
- removed J1, J11, J12, J3-4, J5, J7-8, J9: Conn_01x02, Connector_PinHeader_2.54mm:PinHeader_1x02_P2.54mm_Vertical, symbol Connector_Generic:Conn_01x02
- removed J14: Conn_01x02_Pin, Connector_PinHeader_2.54mm:PinHeader_1x02_P2.54mm_Vertical, symbol Connector:Conn_01x02_Pin
- removed J2, J3: DE9_Plug_MountingHoles, AA_footprints:DSUB-9_Female_Vertical_Pitch2.77x2.84mm_MountingHoles, symbol Connector:DE9_Plug_MountingHoles
- removed J4: Conn_01x03, Connector_PinHeader_2.54mm:PinHeader_1x03_P2.54mm_Vertical, symbol Connector_Generic:Conn_01x03
- removed J7: Conn_01x05, Connector_PinHeader_2.54mm:PinHeader_1x05_P2.54mm_Vertical, symbol Connector_Generic:Conn_01x05
- removed K1, K10, K2, K3, K4, K5, K6, K7, K8, K9: G6E, Relay_THT:Relay_SPDT_Omron_G6E, symbol Relay:G6E
- removed Q1, Q10, Q2, Q3, Q4, Q5, Q6, Q7, Q8, Q9: NMOS, AA_footprints:TO254P470X1016X1965-3P, symbol Simulation_SPICE:NMOS
- removed Q11, Q12: IRLZ44N, Package_TO_SOT_THT:TO-220-3_Vertical, symbol Transistor_FET:IRLZ44N
- removed R1, R29: 4.7k, Resistor_SMD:R_1206_3216Metric_Pad1.30x1.75mm_HandSolder, symbol Device:R
- removed R10, R28, R4, R7: 220, Resistor_SMD:R_1206_3216Metric_Pad1.30x1.75mm_HandSolder, symbol Device:R
- removed R11, R12, R13, R14, R15, R16, R17, R18, R19, R2, R20, R21, R22, R23, R24, R3, R32, R34, R35, R36, R37, R38, R39, R5, R6, R8, R9: 10k, Resistor_SMD:R_1206_3216Metric_Pad1.30x1.75mm_HandSolder, symbol Device:R
- removed R25: 150, Resistor_SMD:R_0805_2012Metric_Pad1.20x1.40mm_HandSolder, symbol Device:R
- removed R26, R27, R40: 1k, Resistor_SMD:R_1206_3216Metric_Pad1.30x1.75mm_HandSolder, symbol Device:R
- removed R30: 60, Resistor_SMD:R_1206_3216Metric_Pad1.30x1.75mm_HandSolder, symbol Device:R
- removed R31, R33: LDR07, OptoDevice:R_LDR_5.1x4.3mm_P3.4mm_Vertical, symbol Sensor_Optical:LDR07
- removed R41: 2,5k, Resistor_SMD:R_1206_3216Metric_Pad1.30x1.75mm_HandSolder, symbol Device:R
- removed R42: 5k, Resistor_SMD:R_1206_3216Metric_Pad1.30x1.75mm_HandSolder, symbol Device:R
- removed R_Shunt1: 5, Resistor_SMD:R_Shunt_Ohmite_LVK12, symbol Device:R_Shunt
- removed SW1, SW2, SW3: SW_DP3T, Button_Switch_THT:SW_DIP_SPSTx02_Piano_10.8x6.64mm_W7.62mm_P2.54mm, symbol Switch:SW_DP3T
- removed SW4, SW7: OP/CL, Button_Switch_SMD:SW_SPST_PTS647_Sx38, symbol Switch:SW_Push
- removed U1: TSR0.5-2450, Converter_DCDC:Converter_DCDC_TRACO_TSR0.5-24xx_TSR0.5-24xxx_THT, symbol Converter_DCDC:TSR0.5-2450
- removed U2: MCP2551-I-SN, Package_SO:SOIC-8_3.9x4.9mm_P1.27mm, symbol Interface_CAN_LIN:MCP2551-I-SN
- removed U4, U5: ${SIM.PARAMS}, AA_footprints:SOT95P280X145-5N, symbol Simulation_SPICE:OPAMP
- removed U6: LM1117DT-3.3, Package_TO_SOT_SMD:TO-252-3_TabPin2, symbol Regulator_Linear:LM1117DT-3.3
- removed Y1: Crystal, Crystal:Crystal_SMD_Abracon_ABM3-2Pin_5.0x3.2mm_HandSoldering, symbol Device:Crystal
Connections:
- no-connect marks 15 -> 0
Other:
- added sheet Alimentació (alimentacio.kicad_sch)
- added sheet Digital (Digital.kicad_sch)
- added sheet Poténcia (Potencia.kicad_sch)
- note removed: "BOTONERA"
- note removed: "BUS CAN"
- note removed: "CALEFACTORS"
- note removed: "CRISTALL"
- note removed: "DRIVER DEL MOTOR DE L'EIX X"
- note removed: "DRIVER DEL MOTOR DE L'EIX Y"
- note removed: "DRIVER DEL MOTOR DE OBRIR I TENCAR"
- note removed: "INPUTS"
- note removed: "LDR'S ANTI-ENLLUERNAMENT"
- note removed: "LEDS SENSOR ANGLE MORT"
- note removed: "Led per a verificar que hi ha corrent."
- note removed: "MICROCONTROLADOR"
- note removed: "REGULADOR DE TENSIÓ"
- note removed: "SENSOR DE CORRENT DE FINAL DE CARRERA"
- note removed: "SW OPEN/CLOSE"
- note removed: "USART"

Commit message: correcions de pcb
Other:
- sheet Poténcia renamed Potencia
Changed lines of the file:
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@@
 	)
 	(sheet
-		(at 19.05 180.34)
-		(size 163.83 82.55)
+		(at 13.97 147.32)
+		(size 213.36 137.16)
 		(exclude_from_sim no)
 		(in_bom yes)
@@
 		)
 		(property "Sheetname" "Digital"
-			(at 53.34 226.06 0)
+			(at 63.754 224.028 0)
 			(effects
 				(font
-					(size 12.7 12.7)
+					(size 17.78 17.78)
 				)
 				(justify left bottom)
@@
 		)
 		(property "Sheetfile" "Digital.kicad_sch"
-			(at 19.05 260.9346 0)
+			(at 13.97 227.9146 0)
 			(effects
 				(font
@@
 		)
 		(property "Field2" ""
-			(at 19.05 180.34 0)
+			(at 13.97 147.32 0)
 			(effects
 				(font
@@
 	(sheet
 		(at 16.51 17.78)
-		(size 146.05 110.49)
+		(size 210.82 129.54)
 		(exclude_from_sim no)
 		(in_bom yes)
@@
 		)
 		(property "Sheetname" "Alimentació"
-			(at 37.338 74.93 0)
+			(at 35.56 90.424 0)
 			(effects
 				(font
-					(size 12.7 12.7)
+					(size 17.78 17.78)
 				)
 				(justify left bottom)
@@
 	)
 	(sheet
-		(at 207.01 41.91)
-		(size 175.26 93.98)
+		(at 228.6 15.24)
+		(size 177.8 237.49)
 		(exclude_from_sim no)
 		(in_bom yes)
 		(on_board yes)
 		(dnp no)
-		(fields_autoplaced yes)
 		(stroke
 			(width 0.2032)
@@
 			(color 0 0 0 0.0000)
 		)
-		(property "Sheetname" "Poténcia"
-			(at 207.01 41.1984 0)
+		(property "Sheetname" "Potencia"
+			(at 259.08 130.81 0)
 			(effects
 				(font
-					(size 1.27 1.27)
+					(size 17.78 17.78)
 				)
 				(justify left bottom)
@@
 		)
 		(property "Sheetfile" "Potencia.kicad_sch"
-			(at 207.01 136.4746 0)
+			(at 228.6 109.8046 0)
 			(effects
 				(font

Commit message: afegit tot final
Other:
- sheet Potencia renamed Potència
Changed lines of the file:
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@@
 		)
 		(property "Sheetname" "Digital"
-			(at 63.754 224.028 0)
+			(at 71.374 221.996 0)
 			(effects
 				(font
 					(size 17.78 17.78)
+					(thickness 3.556)
+					(bold yes)
 				)
 				(justify left bottom)
@@
 				(font
 					(size 17.78 17.78)
+					(thickness 3.556)
+					(bold yes)
 				)
 				(justify left bottom)
@@
 			(color 0 0 0 0.0000)
 		)
-		(property "Sheetname" "Potencia"
+		(property "Sheetname" "Potència"
 			(at 259.08 130.81 0)
 			(effects
 				(font
 					(size 17.78 17.78)
+					(thickness 3.556)
+					(bold yes)
 				)
 				(justify left bottom)
