File: KiCad/Retrovisors_Carlos_Soler_Ingrid_Lopez.kicad_pcb (KiCad board)
At the start: 2 copper layers, 139.2 x 100.5 mm, 127 parts, among them IC1 PIC24H, J1 Conn_01x02, J11 Conn_01x02, J12 Conn_01x02, J14 Conn_01x02_Pin, J2 DE9_Plug_MountingHoles, J3 DE9_Plug_MountingHoles, J3-4 Conn_01x02, J4 Conn_01x03, J5 Conn_01x02, J7 Conn_01x05, J7-8 Conn_01x02, J9 Conn_01x02, K1 G6E, K10 G6E, K2 G6E, K3 G6E, K4 G6E, K5 G6E, K6 G6E, K7 G6E, K8 G6E, K9 G6E, Q1 NMOS, Q10 NMOS, Q11 IRLZ44N, Q12 IRLZ44N, Q2 NMOS, Q3 NMOS, Q4 NMOS, Q5 NMOS, Q6 NMOS, Q7 NMOS, Q8 NMOS, Q9 NMOS, SW1 SW_DP3T, SW2 SW_DP3T, SW3 SW_DP3T, SW4 OP/CL, SW7 OP/CL, U1 TSR0.5-2450, U2 MCP2551-I-SN, U3 PCF8574P, U4 type="X" model="OPAMP" lib="", U5 type="X" model="OPAMP" lib="", U6 LM1117DT-3.3, Y1 Crystal

Commit message: canvis pcb finals
Parts:
- moved SW2 84.4 mm to (169.7, 65.8), turned to 0 degrees
- moved C7 72.6 mm to (163.3, 133.0), turned to -90 degrees
- moved R3 70.0 mm to (163.1, 68.6)
- moved R2 68.9 mm to (163.1, 64.5)
- moved R4 68.9 mm to (176.3, 72.1)
- moved SW3 68.3 mm to (169.8, 78.5), turned to 0 degrees
- moved TP2 68.0 mm to (148.3, 120.5)
- moved TP1 67.6 mm to (160.3, 121.0)
- moved R8 63.4 mm to (168.1, 72.1)
- moved R10 62.0 mm to (176.3, 74.7)
- moved R9 59.2 mm to (171.2, 74.7), turned to 180 degrees
- moved SW1 50.9 mm to (169.8, 93.7), turned to 0 degrees
- moved R5 45.8 mm to (170.7, 88.4), turned to 0 degrees
- moved R6 45.7 mm to (173.7, 85.9), turned to 180 degrees
- moved R7 44.1 mm to (176.8, 88.4)
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Connections:
- D11 pad 2: /Potencia/Vdrain3 -> /Potencia/Vdrain8
- D12 pad 2: /Potencia/Vdrain1 -> /Potencia/Vdrain9
- D13 pad 2: /Potencia/Vdrain2 -> /Potencia/Vdrain10
- D3 pad 2: /Potencia/Vdrain4 -> /Potencia/Vdrain3
- D4 pad 2: /Potencia/Vdrain3 -> /Potencia/Vdrain4
- D8 pad 2: /Potencia/Vdrain1 -> /Potencia/Vdrain5
- D9 pad 2: /Potencia/Vdrain4 -> /Potencia/Vdrain7
- IC1 pad 12: SC_IN -> unconnected-(IC1-RC1/T1OSI-Pad12)
- IC1 pad 16: unconnected-(IC1-RC5/SDO-Pad16) -> SC_IN
- IC1 pad 2: CAL_L -> Net-(IC1-RA0/AN0)
- IC1 pad 23: CANTX -> CANRX
- IC1 pad 24: CANRX -> CANTX
- IC1 pad 3: CAL_R -> Net-(IC1-RA1/AN1)
- IC1 pad 4: Net-(IC1-RA2/AN2/VREF-) -> CAL_R
- IC1 pad 5: Net-(IC1-RA3/AN3/VREF+) -> CAL_L
- J4 pad 2: MCLR -> reset
- J4 pad 3: reset -> MCLR
- K10 pad 6: /Potencia/Vdrain2 -> /Potencia/Vdrain10
- K3 pad 6: /Potencia/Vdrain4 -> /Potencia/Vdrain3
- K4 pad 6: /Potencia/Vdrain3 -> /Potencia/Vdrain4
- K5 pad 6: /Potencia/Vdrain1 -> /Potencia/Vdrain5
- K7 pad 6: /Potencia/Vdrain4 -> /Potencia/Vdrain7
- K8 pad 6: /Potencia/Vdrain3 -> /Potencia/Vdrain8
- K9 pad 6: /Potencia/Vdrain1 -> /Potencia/Vdrain9
- Q10 pad 1: /Potencia/Vdrain2 -> /Potencia/Vdrain10
- Q3 pad 1: /Potencia/Vdrain4 -> /Potencia/Vdrain3
- Q4 pad 1: /Potencia/Vdrain3 -> /Potencia/Vdrain4
- Q5 pad 1: /Potencia/Vdrain1 -> /Potencia/Vdrain5
- Q7 pad 1: /Potencia/Vdrain4 -> /Potencia/Vdrain7
- Q8 pad 1: /Potencia/Vdrain3 -> /Potencia/Vdrain8
- Q9 pad 1: /Potencia/Vdrain1 -> /Potencia/Vdrain9
- R31 pad 2: Net-(IC1-RA2/AN2/VREF-) -> Net-(IC1-RA0/AN0)
- R32 pad 1: Net-(IC1-RA2/AN2/VREF-) -> Net-(IC1-RA0/AN0)
- R33 pad 2: Net-(IC1-RA3/AN3/VREF+) -> Net-(IC1-RA1/AN1)
- R34 pad 1: Net-(IC1-RA3/AN3/VREF+) -> Net-(IC1-RA1/AN1)
- R40 pad 2: Net-(U5-V-) -> GND
- R42 pad 1: Net-(U5-V-) -> GND
- U3 pad 5: DLY_U -> DM_C
- U3 pad 6: DM_O -> DLY_U
- U3 pad 7: DM_C -> DM_O
- U5 pad 5: Net-(U5-V-) -> GND
Routing:
- net GND: track 167.3 -> 48.0 mm, vias 117 -> 172
- net /Potencia/Vdrain2: track 73.5 -> 11.2 mm, vias 1 -> 0
- net /Potencia/Vdrain1: track 95.6 -> 41.7 mm, vias 1 -> 0
- net /Potencia/Vdrain3: track 54.3 -> 11.4 mm
- net /Potencia/Vdrain4: track 52.0 -> 10.5 mm
- net Net-(IC1-RA0/AN0): track 0.00 -> 35.5 mm
- net Net-(IC1-RA1/AN1): track 0.00 -> 29.9 mm
- net DLY_U: track 53.5 -> 78.5 mm
- net Net-(IC1-RC4/SDI/SDA): track 41.1 -> 62.7 mm, vias 1 -> 2
- net DLX_U: track 61.0 -> 39.9 mm
- net Net-(J4-Pin_1): track 20.4 -> 0.56 mm
- net Net-(IC1-RA2/AN2/VREF-): track 19.4 -> 0.00 mm
- net Net-(IC1-RA3/AN3/VREF+): track 14.2 -> 0.00 mm
- net RM_button: track 48.3 -> 34.3 mm, vias 0 -> 1
- net reset: track 27.3 -> 13.9 mm
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Other:
- board size 139.2 x 100.5 mm -> 143.5 x 100.8 mm

Commit message: pcb definitiva
Parts:
- moved R43 33.4 mm to (126.3, 125.4), turned to -90 degrees
- moved R44 27.8 mm to (126.2, 120.3), turned to -90 degrees
- moved R26 22.5 mm to (164.0, 128.9), turned to 180 degrees
- moved U3 19.4 mm to (133.6, 116.2), turned to 180 degrees
- moved R27 15.3 mm to (158.8, 131.1)
- moved R35 13.6 mm to (149.0, 126.6)
- moved SW7 13.6 mm to (143.3, 126.6)
- moved D2 12.7 mm to (158.8, 126.0), turned to 0 degrees
- moved D7 12.7 mm to (158.8, 128.2), turned to 180 degrees
- moved J3 7.74 mm to (186.0, 112.6)
- moved J2 7.38 mm to (188.9, 91.7)
- moved R36 6.48 mm to (153.2, 141.0)
- moved REF** 5.55 mm to (188.4, 141.8)
- moved REF** 4.23 mm to (54.7, 141.8)
- moved R28 4.04 mm to (154.3, 124.6)
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Connections:
- net /Digital/osc1 renamed /Digital/OSC1
- net /Digital/osc2 renamed /Digital/OSC2
- net Net-(D1-A) renamed /Alimentació/LD_V
- net Net-(D10-A) renamed /Potencia/Vdrain6
- net Net-(D2-A) renamed /Alimentació/ALD2
- net Net-(D2-K) renamed /Alimentació/ALD1
- net Net-(IC1-RA0/AN0) renamed /Digital/AL1
- net Net-(IC1-RA1/AN1) renamed /Digital/AL2
- net Net-(IC1-RC0/T1OSO/T13CKI) renamed /Digital/SP
- net Net-(IC1-RC3/SCK/SCL) renamed /Digital/SCL
- net Net-(IC1-RC4/SDI/SDA) renamed /Digital/SDA
- net Net-(J4-Pin_1) renamed /Digital/ConMu
- net Net-(R2-Pad1) renamed /Digital/LM_BO
- net Net-(R36-Pad1) renamed /Potencia/RSH2
- net Net-(R37-Pad1) renamed /Potencia/RSH3
- net Net-(R5-Pad1) renamed /Digital/RM_BO
- net Net-(R8-Pad1) renamed /Digital/SE_BO
- net Net-(U1-Vout) renamed /Alimentació/V_Buck
- net Net-(U2-Rs) renamed /Digital/RS
- net Net-(U4-+) renamed /Potencia/O1V+
- net Net-(U4--) renamed /Potencia/O1V-
- net Net-(U5-+) renamed /Potencia/O2V+
- net Net-(U5--) renamed /Potencia/O2V-
- U3 pad 12: DLX_D -> DRX_U
- U3 pad 9: DRX_U -> DLX_D
Routing:
- net DLX_U: track 39.9 -> 104.6 mm, vias 2 -> 0
- net DRX_D: track 9.72 -> 60.9 mm
- net DRX_U: track 32.3 -> 77.5 mm, vias 1 -> 0
- net DM_O: track 12.3 -> 50.1 mm
- net /Potencia/Vdrain1: track 41.7 -> 11.3 mm
- net DLX_D: track 57.2 -> 86.5 mm
- net GND: track 48.0 -> 29.5 mm, vias 172 -> 177
- net /Digital/SDA: track 62.7 -> 51.0 mm, vias 2 -> 1
- net VBAT_PROT: track 0.18 -> 11.3 mm
- net DLY_D: track 65.9 -> 76.6 mm
- net /Potencia/O1V+: track 3.27 -> 11.3 mm
- net DM_C: track 37.2 -> 44.2 mm
- net /Potencia/RSH2: track 15.6 -> 8.75 mm
- net /Digital/CAN+: track 19.0 -> 25.3 mm
- net /Digital/RM_BO: track 4.35 -> 9.94 mm
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Other:
- board size 143.5 x 100.8 mm -> 144.1 x 99 mm

Commit message: placa definitivisima
Parts:
- moved J3 28.1 mm to (174.0, 138.0), turned to 0 degrees
- moved J2 21.8 mm to (188.5, 113.5)
- moved SW1 21.0 mm to (190.0, 88.0), turned to 180 degrees
- moved SW2 20.9 mm to (190.0, 70.5), turned to 180 degrees
- moved SW3 20.2 mm to (190.0, 79.5), turned to 180 degrees
- moved R36 16.4 mm to (137.0, 138.0)
- moved R_Shunt1 13.3 mm to (133.9, 135.0)
- moved R37 13.3 mm to (137.0, 132.0)
- moved R39 13.3 mm to (141.5, 133.5)
- moved U4 13.3 mm to (145.1, 134.0)
- moved R38 12.6 mm to (150.0, 134.0)
- moved R3 10.4 mm to (173.5, 68.0), turned to 180 degrees
- moved R2 9.54 mm to (170.5, 70.5)
- moved R42 8.02 mm to (174.5, 129.0)
- moved R41 7.55 mm to (174.5, 124.0)
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Routing:
- net GND: track 29.5 -> 9.44 mm, vias 177 -> 187
- net /Digital/SE_BO: track 6.45 -> 24.2 mm
- net /Digital/RM_BO: track 9.94 -> 27.5 mm
- net /Potencia/O2V+: track 13.3 -> 30.4 mm
- net /Digital/RX: track 22.3 -> 35.7 mm
- net FI_MOTOR: track 83.5 -> 71.2 mm
- net /Digital/TX: track 22.9 -> 35.2 mm
- net /Digital/LM_BO: track 9.65 -> 0.00 mm
- net /Digital/CAN+: track 25.3 -> 15.7 mm
- net /Digital/CAN-: track 26.0 -> 17.1 mm
- net /Digital/SP: track 22.7 -> 14.6 mm
- net SC_IN: track 18.8 -> 14.6 mm
- net RM_button: track 32.8 -> 36.5 mm, vias 1 -> 2
- net /Potencia/RSH2: track 8.75 -> 5.59 mm
- net LM_button: track 46.1 -> 48.9 mm
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
Commit message: diseny final final
Parts:
- moved R41 5.00 mm to (174.5, 129.0), turned to -90 degrees
- moved R42 5.00 mm to (174.5, 124.0), turned to -90 degrees
- moved TP3 2.21 mm to (159.0, 121.0)
Routing:
- net /Digital/LM_BO: track 0.00 -> 23.5 mm
- net /Digital/SP: track 14.6 -> 22.0 mm
- net FI_MOTOR: track 71.2 -> 68.7 mm
- net angle_m: track 8.64 -> 9.48 mm

Commit message: afegit tot final
Parts:
- J7-8: value Conn_01x02 -> J1
Other:
- board text added: "29/04/2026"
- board text added: "ANGLE-MORT"
- board text added: "ANTI-ATRAPAMENT"
- board text added: "ANTI-ENLLUERNAMENT"
- board text added: "BUS CAN"
- board text added: "CALEFACTORS"
- board text added: "CONNEXIÓ BATERIA"
- board text added: "DRIVERS DE MOTOR"
- board text added: "Ingrid Lopez- Carlos Soler"
- board text added: "Ingrid Lopez-Carlos Soler Miralls d'un cotxe"
- board text added: "OP/CL"
- board text added: "PCB RETROVISORS D'UN COTXE"
- board text added: "REGULADOR DE TENSIÓ"
- board text added: "SWITCHES"
- board text added: "USART"
