File: KiCad/alimentacio.kicad_sch (KiCad schematic)
At the start: 20 parts, among them J14 Conn_01x02_Pin, U1 TSR0.5-2450, U6 LM1117DT-3.3

Commit message: pcb definitiva
Connections:
- net ALD1: now reaches D2.1 (K), D7.2 (A), R28.1
- net ALD2: now reaches D2.2 (A), D7.1 (K), R26.2, R27.1
- net V_Buck: now reaches C10.1, C11.1, C12.1, C13.1, U1.3 (Vout), U6.3 (VI)
- net LD_V: now reaches D1.2 (A), R25.2
Other:
- note added: "25/05/2026"
- note added: "Alimentació del Retrovisor"
- note added: "Aqui podem veure com pasem de la tensio de la bateria (12V) a la Tensio de 3.3V"
Changed lines of the file:
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@@
+		)
+	)
+	(text "25/05/2026\n"
+		(exclude_from_sim no)
+		(at 212.598 193.802 0)
+		(effects
+			(font
+				(size 1.27 1.27)
+			)
 		)
 	)
@@
 		)
 	)
+	(text "Aqui podem veure com pasem de la tensio de la bateria (12V)\n a la Tensio de 3.3V"
+		(exclude_from_sim no)
+		(at 179.07 169.672 0)
+		(effects
+			(font
+				(size 1.27 1.27)
+			)
+			(justify left)
+		)
+	)
+	(text "Alimentació del Retrovisor\n"
+		(exclude_from_sim no)
+		(at 198.882 189.484 0)
+		(effects
+			(font
+				(size 1.27 1.27)
+			)
+		)
+	)
 	(junction
 		(at 107.95 24.13)
@@
 	)
 	(junction
-		(at 40.64 40.64)
-		(diameter 0)
-		(color 0 0 0 0)
-	)
-	(junction
 		(at 135.89 43.18)
 		(diameter 0)
@@
 	(wire
 		(pts
+			(xy 226.06 54.61) (xy 228.6 54.61)
+		)
+		(stroke
+			(width 0)
+			(type default)
+		)
+	)
+	(wire
+		(pts
+			(xy 39.37 38.1) (xy 34.29 38.1)
+		)
+		(stroke
+			(width 0)
+			(type default)
+		)
+	)
+	(wire
+		(pts
 			(xy 118.11 24.13) (xy 118.11 26.67)
 		)
@@
 	(wire
 		(pts
-			(xy 34.29 38.1) (xy 39.624 38.1)
-		)
-		(stroke
-			(width 0)
-			(type default)
-		)
-	)
-	(wire
-		(pts
 			(xy 240.03 55.88) (xy 240.03 58.42)
 		)
@@
 	(wire
 		(pts
-			(xy 40.64 40.64) (xy 40.894 40.64)
-		)
-		(stroke
-			(width 0)
-			(type default)
-		)
-	)
-	(wire
-		(pts
 			(xy 50.8 24.13) (xy 54.61 24.13)
 		)
@@
 	(wire
 		(pts
-			(xy 228.6 54.61) (xy 226.06 54.61)
+			(xy 36.83 105.41) (xy 36.83 107.95)
 		)
 		(stroke
@@
 	(wire
 		(pts
+			(xy 39.37 43.18) (xy 39.37 40.64)
+		)
+		(stroke
+			(width 0)
+			(type default)
+		)
+	)
+	(wire
+		(pts
 			(xy 135.89 24.13) (xy 140.97 24.13)
 		)
@@
 	(wire
 		(pts
-			(xy 34.29 40.64) (xy 40.64 40.64)
-		)
-		(stroke
-			(width 0)
-			(type default)
-		)
-	)
-	(wire
-		(pts
 			(xy 127 24.13) (xy 135.89 24.13)
 		)
@@
 	(wire
 		(pts
+			(xy 236.22 58.42) (xy 240.03 58.42)
+		)
+		(stroke
+			(width 0)
+			(type default)
+		)
+	)
+	(wire
+		(pts
 			(xy 107.95 44.45) (xy 114.3 44.45)
 		)
@@
 	(wire
 		(pts
-			(xy 236.22 58.42) (xy 240.03 58.42)
-		)
-		(stroke
-			(width 0)
-			(type default)
-		)
-	)
-	(wire
-		(pts
 			(xy 93.98 44.45) (xy 77.47 44.45)
 		)
@@
 	(wire
 		(pts
+			(xy 39.37 36.83) (xy 39.37 38.1)
+		)
+		(stroke
+			(width 0)
+			(type default)
+		)
+	)
+	(wire
+		(pts
 			(xy 127 43.18) (xy 135.89 43.18)
 		)
@@
 	(wire
 		(pts
-			(xy 36.83 105.41) (xy 36.83 107.95)
-		)
-		(stroke
-			(width 0)
-			(type default)
-		)
-	)
-	(wire
-		(pts
 			(xy 135.89 33.02) (xy 135.89 43.18)
 		)
@@
 			(width 0)
 			(type default)
+		)
+	)
+	(wire
+		(pts
+			(xy 39.37 40.64) (xy 34.29 40.64)
+		)
+		(stroke
+			(width 0)
+			(type default)
+		)
+	)
+	(wire
+		(pts
+			(xy 220.98 66.04) (xy 220.98 67.31)
+		)
+		(stroke
+			(width 0)
+			(type default)
+		)
+	)
+	(label "ALD2"
+		(at 228.6 54.61 90)
+		(effects
+			(font
+				(size 1.27 1.27)
+			)
+			(justify left bottom)
+		)
+	)
+	(label "V_Buck"
+		(at 129.54 24.13 90)
+		(effects
+			(font
+				(size 1.27 1.27)
+			)
+			(justify left bottom)
+		)
+	)
+	(label "ALD1"
+		(at 238.76 58.42 270)
+		(effects
+			(font
+				(size 1.27 1.27)
+			)
+			(justify right bottom)
+		)
+	)
+	(label "LD_V"
+		(at 36.83 96.52 180)
+		(effects
+			(font
+				(size 1.27 1.27)
+			)
+			(justify right bottom)
 		)
 	)
@@
 	)
 	(symbol
+		(lib_id "power:+12V")
+		(at 39.37 36.83 0)
+		(unit 1)
+		(exclude_from_sim no)
+		(in_bom yes)
+		(on_board yes)
+		(dnp no)
+		(property "Reference" "#PWR031"
+			(at 39.37 40.64 0)
+			(effects
+				(font
+					(size 1.27 1.27)
+				)
+				(hide yes)
+			)
+		)
+		(property "Value" "+12V"
+			(at 36.703 33.2232 0)
+			(effects
+				(font
+					(size 1.27 1.27)
+				)
+				(justify left)
+			)
+		)
+		(property "Footprint" ""
+			(at 39.37 36.83 0)
+			(effects
+				(font
+					(size 1.27 1.27)
+				)
+				(hide yes)
+			)
+		)
+		(property "Datasheet" ""
+			(at 39.37 36.83 0)
+			(effects
+				(font
+					(size 1.27 1.27)
+				)
+				(hide yes)
+			)
+		)
+		(property "Description" ""
+			(at 39.37 36.83 0)
+			(effects
+				(font
+					(size 1.27 1.27)
+				)
+			)
+		)
+		(pin "1"
+		)
+		(instances
+			(project "Retrovisors_Carlos_Soler_Ingrid_Lopez"
+				(path "/a9cf8edd-cd44-4958-b775-951afc8c27af/b8e06db1-76a8-45c4-8cb5-d5e2adcbfa40"
+					(reference "#PWR031")
+					(unit 1)
+				)
+			)
+		)
+	)
+	(symbol
 		(lib_id "Device:C")
 		(at 67.31 30.48 0)
@@
 	(symbol
 		(lib_id "power:GND")
-		(at 40.64 40.64 0)
+		(at 39.37 43.18 0)
 		(unit 1)
 		(exclude_from_sim no)
@@
 		(fields_autoplaced yes)
 		(property "Reference" "#PWR078"
-			(at 40.64 46.99 0)
+			(at 39.37 49.53 0)
 			(effects
 				(font
@@
 		)
 		(property "Value" "GND"
-			(at 40.64 45.72 0)
+			(at 39.37 48.26 0)
 			(effects
 				(font
@@
 		)
 		(property "Footprint" ""
-			(at 40.64 40.64 0)
+			(at 39.37 43.18 0)
 			(effects
 				(font
@@
 		)
 		(property "Datasheet" ""
-			(at 40.64 40.64 0)
+			(at 39.37 43.18 0)
 			(effects
 				(font
@@
 		)
 		(property "Description" "Power symbol creates a global label with name \"GND\" , ground"
-			(at 40.64 40.64 0)
+			(at 39.37 43.18 0)
 			(effects
 				(font
@@
 		(lib_name "GND_2")
 		(lib_id "power:GND")
-		(at 220.98 66.04 0)
+		(at 220.98 67.31 0)
 		(unit 1)
 		(exclude_from_sim no)
@@
 		(dnp no)
 		(property "Reference" "#PWR019"
-			(at 220.98 72.39 0)
+			(at 220.98 73.66 0)
 			(effects
 				(font
@@
 		)
 		(property "Value" "GND"
-			(at 225.298 66.04 0)
+			(at 225.298 67.31 0)
 			(effects
 				(font
@@
 		)
 		(property "Footprint" ""
-			(at 220.98 66.04 0)
+			(at 220.98 67.31 0)
 			(effects
 				(font
@@
 		)
 		(property "Datasheet" ""
-			(at 220.98 66.04 0)
+			(at 220.98 67.31 0)
 			(effects
 				(font
@@
 		)
 		(property "Description" "Power symbol creates a global label with name \"GND\" , ground"
-			(at 220.98 66.04 0)
+			(at 220.98 67.31 0)
 			(effects
 				(font
@@
 					(unit 1)
 				)
-			)
-		)
-	)
-	(symbol
-		(lib_id "power:+12V")
-		(at 39.624 38.1 0)
-		(unit 1)
-		(exclude_from_sim no)
-		(in_bom yes)
-		(on_board yes)
-		(dnp no)
-		(fields_autoplaced yes)
-		(property "Reference" "#PWR057"
-			(at 39.624 41.91 0)
-			(effects
-				(font
-					(size 1.27 1.27)
-				)
-				(hide yes)
-			)
-		)
-		(property "Value" "+12V"
-			(at 42.164 37.465 0)
-			(effects
-				(font
-					(size 1.27 1.27)
-				)
-				(justify left)
-			)
-		)
-		(property "Footprint" ""
-			(at 39.624 38.1 0)
-			(effects
-				(font
-					(size 1.27 1.27)
-				)
-				(hide yes)
-			)
-		)
-		(property "Datasheet" ""
-			(at 39.624 38.1 0)
-			(effects
-				(font
-					(size 1.27 1.27)
-				)
-				(hide yes)
-			)
-		)
-		(property "Description" ""
-			(at 39.624 38.1 0)
-			(effects
-				(font
-					(size 1.27 1.27)
-				)
-			)
-		)
-		(pin "1"
-		)
-		(instances
-			(project "Retrovisors_Carlos_Soler_Ingrid_Lopez"
-				(path "/a9cf8edd-cd44-4958-b775-951afc8c27af/b8e06db1-76a8-45c4-8cb5-d5e2adcbfa40"
-					(reference "#PWR057")
-					(unit 1)
-				)

Commit message: afegit tot final
Other:
- moved on the sheet: D1, D2, D7, R25, R26, R27, R28
